Commit message: feat: add use_sn_prefix to decouple joint names from robot_sn
`compute_arm_prefix` builds the joint/link prefix as `arm_prefix + robot_sn`,
which conflates two unrelated things. `robot_sn` is how the RDK addresses the arm
— it must be a real serial, and `ros2 launch` rejects an empty one. The prefix is
a naming namespace. `flexiv.ros2_control.xacro` already takes them as separate
hardware params, so the coupling exists only in the name.

Coupling them forces every consumer to know the serial: the joint list in
`flexiv_controllers.yaml`, MoveIt's joint limits, and every joint name in a
downstream stack, which turns otherwise arm-generic config into per-arm config.

`use_sn_prefix` (default true) makes this opt-in rather than changing behaviour:

  use_sn_prefix:=true   (default)  Enlight-L-000000_joint1   <- unchanged
  use_sn_prefix:=false             joint1

The prefix is now assembled by joining the non-empty components, so neither
setting can produce a leading or doubled underscore, and an all-empty result is
still the empty string — which `mico_core.xacro` relies on for `torso_base_link`.

Wired into the single-arm branch only. Dual-arm, paired, and AICO branches
disambiguate with explicit `left`/`right` prefixes and are untouched.

Verified with flexiv_ros2 v2.2's `flexiv_hardware/urdf/flexiv.urdf.xacro`:
  - default and use_sn_prefix:=true  -> Enlight-L-000000_joint1
  - use_sn_prefix:=false, mock + real -> joint1, ros2_control block present
  - real hardware still gets <param name="robot_sn">Enlight-L-000000</param>
  - no leading or doubled underscores in any name
  - dual arm (Enlight-LL) -> left_joint1 / right_joint1, unchanged

File: urdf/common/flexiv_common.xacro (robot description, xacro)
@@ -5,10 +5,27 @@
     'computed_arm_prefix'.
     This is the single source of truth for the prefix.
-    arm_prefix: 'left', 'right' or '' (user-supplied prefixes also allowed)
-    robot_sn:   robot serial number, may be empty
-  -->
-  <xacro:macro name="compute_arm_prefix" params="arm_prefix:='' robot_sn:=''">
+    arm_prefix:    'left', 'right' or '' (user-supplied prefixes also allowed)
+    robot_sn:      robot serial number, may be empty
+    use_sn_prefix: whether `robot_sn` contributes to joint and link names
+    `use_sn_prefix` defaults to true, which is the historical behaviour:
+    `<arm_prefix>_<robot_sn>_`, or `<robot_sn>_` when `arm_prefix` is empty.
+    Set it false to name joints and links from `arm_prefix` alone, leaving
+    `robot_sn` to do only what it must — address the arm over the RDK. The two are
+    otherwise independent (`flexiv.ros2_control.xacro` already takes `robot_sn` and
+    `prefix` as separate hardware params), but coupling them in the name forces
+    every consumer to know the serial: the joint list in
+    `flexiv_controllers.yaml`, MoveIt's joint limits, and every joint name in a
+    downstream stack, which turns otherwise arm-generic config into per-arm
+    config. `robot_sn` also cannot simply be emptied to avoid this — `ros2 launch`
+    rejects an empty value, and the hardware interface needs a real serial.
+    Either way the result has no leading or doubled underscore: each present
+    component contributes exactly one trailing separator, and an all-empty result
+    is the empty string rather than '_' (see the `torso_base_link` note in
+    `mico_core.xacro`, which depends on this).
+  -->
+  <xacro:macro name="compute_arm_prefix" params="arm_prefix:='' robot_sn:='' use_sn_prefix:=true">
+    <xacro:property name="sn_part" value="${robot_sn if use_sn_prefix else ''}" lazy_eval="false" />
     <xacro:property name="computed_arm_prefix"
-      value="${(arm_prefix + '_' + robot_sn + '_') if arm_prefix != '' and robot_sn != '' else (arm_prefix + robot_sn + '_') if (arm_prefix + robot_sn) != '' else ''}"
+      value="${''.join([part + '_' for part in [arm_prefix, sn_part] if part != ''])}"
       scope="parent" />
   </xacro:macro>

File: urdf/common/flexiv_robot.xacro (robot description, xacro)
@@ -10,4 +10,5 @@
     visual_parameters_file
     arm_prefix:=''
+    use_sn_prefix:=true
     load_gripper:=false
     gripper_name:='Flexiv-GN01'
@@ -19,5 +20,6 @@
     ">
     <xacro:include filename="$(find flexiv_description)/urdf/common/flexiv_common.xacro" />
-    <xacro:compute_arm_prefix arm_prefix="${arm_prefix}" robot_sn="${robot_sn}" />
+    <xacro:compute_arm_prefix arm_prefix="${arm_prefix}" robot_sn="${robot_sn}"
+      use_sn_prefix="${use_sn_prefix}" />
     <xacro:property name="prefix" value="${computed_arm_prefix}" />
     <xacro:if value="${load_gripper and gripper_name=='Flexiv-GN01'}">

File: urdf/flexiv.urdf.xacro (robot description, xacro)
@@ -24,4 +24,13 @@
   <!-- parameters -->
   <xacro:arg name="arm_prefix" default="" />
+  <!--
+    Whether `robot_sn` contributes to joint and link names. True keeps the
+    historical `<robot_sn>_joint1` naming; false names joints from `arm_prefix`
+    alone and leaves `robot_sn` to address the arm over the RDK. See
+    `compute_arm_prefix` in `urdf/common/flexiv_common.xacro`.
+    Wired into the single-arm branch only. The dual-arm, paired, and AICO branches
+    disambiguate with explicit `left`/`right` prefixes and are unaffected.
+  -->
+  <xacro:arg name="use_sn_prefix" default="true" />
   <xacro:arg name="robot_sn" default="" />
   <xacro:arg name="joint_limits_parameters_file"
@@ -88,4 +97,5 @@
       visual_parameters_file="$(arg visual_parameters_file)"
       arm_prefix="$(arg arm_prefix)"
+      use_sn_prefix="$(arg use_sn_prefix)"
       load_gripper="$(arg load_gripper)"
       gripper_name="$(arg gripper_name)"
