Commit message: fix(enlight): Take upstream's Enlight-L model fixes
The Enlight-L parts of flexivrobotics/flexiv_description d0ece5a
("Backport/Fix mesh xacro and update robot model data (#40)",
2026-10-19), which upstream carries on humble, jazzy and lyrical but
not on the humble-v2 release line this branch tracks:

- `get_inertias` wraps its origin, mass and inertia in `<inertial>`.
  urdfdom reads mass only from that element, so without it every
  arm link was massless to any consumer that builds dynamics from the
  description (MoveIt's KDL chain, and so chef's ITLP torque checks):
  a rendered Enlight-LL had 0 `<inertial>` blocks and 16 bare `<mass>`
  tags.
- Enlight-L joint velocity limits: joints 1-4 2.0944 -> 2.4958 rad/s,
  joints 5-7 6.0214 -> 5.4105 rad/s.
- The Enlight-L visual meshes reference their `linkN.mtl` files by the
  lowercase names they ship with.

Left out of the same upstream commit: the MICO, AICO and Rizon configs
and meshes, the README, and the optional soft-limits branch of
`get_joint_limits`, which only the MICO torso joints need.

Rendered Enlight-LL with xacro from this tree: 16 links with
`<inertial>` (two arms, base through link7), 30.72 kg in total,
8 joints at 2.4958 and 6 at 5.4105 rad/s; `check_urdf` parses it.

Co-authored-by: Claude Fable 5.1 <noreply@anthropic.com>

File: urdf/common/flexiv_common.xacro (robot description, xacro)
@@ -94,11 +94,13 @@
   <xacro:macro name="get_inertias" params="name">
     <xacro:property name="inertias" value="${sec_inertia_parameters[name]}" lazy_eval="false" />
-    <origin xyz="${inertias['origin']['x']} ${inertias['origin']['y']} ${inertias['origin']['z']}"
-      rpy="${inertias['origin']['roll']} ${inertias['origin']['pitch']} ${inertias['origin']['yaw']}" />
-    <mass value="${inertias['mass']}" />
-    <inertia ixx="${inertias['inertia']['ixx']}" ixy="${inertias['inertia']['ixy']}"
-      ixz="${inertias['inertia']['ixz']}" iyy="${inertias['inertia']['iyy']}"
-      iyz="${inertias['inertia']['iyz']}"
-      izz="${inertias['inertia']['izz']}" />
+    <inertial>
+      <origin xyz="${inertias['origin']['x']} ${inertias['origin']['y']} ${inertias['origin']['z']}"
+        rpy="${inertias['origin']['roll']} ${inertias['origin']['pitch']} ${inertias['origin']['yaw']}" />
+      <mass value="${inertias['mass']}" />
+      <inertia ixx="${inertias['inertia']['ixx']}" ixy="${inertias['inertia']['ixy']}"
+        ixz="${inertias['inertia']['ixz']}" iyy="${inertias['inertia']['iyy']}"
+        iyz="${inertias['inertia']['iyz']}"
+        izz="${inertias['inertia']['izz']}" />
+    </inertial>
   </xacro:macro>
   <!--
