Commit message: feat: armN prefixes, use_sn_prefix, and per-arm initial positions
Backport of chef's fork features onto humble-v2.1, which is the release that
pairs with RDK v2.1 and Enlight software v3E.1. The previous fork branch sat
on the consolidated `humble` line, whose RDK v2.2 requirement is what made it
incompatible with the robot's firmware.

Three changes, all so a consumer can model a dual-arm Enlight-LL with joint
names it can write into its own SRDF, limits and controller config:

  - `use_sn_prefix` (default `true`, i.e. upstream behaviour) decouples
    link/joint names from `robot_sn`. Upstream builds the prefix as
    `<arm_prefix>_<robot_sn>_`, which forces a per-robot regeneration of every
    downstream file that names a joint. `robot_sn` still reaches the RDK
    separately; it is how the robot is addressed and stays a real serial.

  - the dual branch uses `arm1`/`arm2` rather than `left`/`right`, so the two
    arms are numbered rather than sided. Sidedness is a property of the
    mounting, not of the kinematic chain.

  - per-arm initial positions. Upstream feeds both arms one file, so a
    consumer that plans a single arm cannot seed a start pose for it without
    also moving the other. Only mock hardware reads these; a real arm reports
    its own joints.

The `<ros2_control>` prefixes are now DERIVED rather than hardcoded, which is
the load-bearing part. Upstream writes `prefix_left="left_$(arg robot_sn)_"`
inline, so any change to `arm_prefix` or `use_sn_prefix` silently desyncs the
`<joint>` names inside `<ros2_control>` from the ones in the link tree. The
result expands fine and then leaves the controller unable to claim its
interfaces, showing up only as a controller that never reaches `active`.

Verified by expanding the URDF and cross-checking both joint-name sets:

  LL sn_prefix=false: 14 tree joints, 14 ros2_control joints, mismatch=none
  LL sn_prefix=true : 14 tree joints, 14 ros2_control joints, mismatch=none
  L  sn_prefix=false:  7 tree joints,  7 ros2_control joints, mismatch=none
  L  sn_prefix=true :  7 tree joints,  7 ros2_control joints, mismatch=none

and per-arm seeding: arm1_joint4=1.1 (override) vs arm2_joint4=1.570796
(vendor default).

Co-Authored-By: Claude Opus 5 (1M context) <noreply@anthropic.com>

File: urdf/common/enlight_robot.xacro (robot description, xacro)
@@ -10,4 +10,5 @@
     visual_parameters_file
     arm_prefix:=''
+    use_sn_prefix:=true
     load_gripper:=false
     gripper_name:='Flexiv-GN01'
@@ -23,6 +24,16 @@
     base_rpy:='0.0 0.0 0.0'
     ">
+    <!--
+      Link/joint name prefix, built from the non-empty parts of
+      `arm_prefix` and (optionally) `robot_sn`, each followed by `_`.
+      `use_sn_prefix:=false` drops the serial, which is what lets a
+      consumer name joints `arm1_joint1..7` instead of
+      `arm1_<serial>_joint1..7`. `robot_sn` still reaches the RDK
+      separately (it is how the robot is addressed and must stay a real
+      serial), so this only decouples the joint *names* from it.
+    -->
+    <xacro:property name="sn_part" value="${robot_sn if use_sn_prefix else ''}" lazy_eval="false" />
     <xacro:property name="prefix"
-      value="${(arm_prefix + '_' + robot_sn + '_') if arm_prefix != '' and robot_sn != '' else (arm_prefix + robot_sn + '_') if (arm_prefix + robot_sn) != '' else ''}" />
+      value="${''.join([part + '_' for part in [arm_prefix, sn_part] if part != ''])}" />
     <xacro:property name="load_mounted_ft_sensor" value="false" />
     <xacro:if value="${load_gripper and gripper_name=='Flexiv-GN01'}">

File: urdf/flexiv.urdf.xacro (robot description, xacro)
@@ -13,4 +13,12 @@
   <!-- parameters -->
   <xacro:arg name="arm_prefix" default="" />
+  <!--
+    Whether `robot_sn` becomes part of link/joint names. Upstream default is
+    `true` (`arm1_<serial>_joint1`); `false` gives bare `arm1_joint1`, which is
+    what a consumer wants when its own config, SRDF and limits name joints
+    without a per-robot serial in them. `robot_sn` still reaches the RDK either
+    way, since that is how the robot is addressed.
+  -->
+  <xacro:arg name="use_sn_prefix" default="true" />
   <xacro:arg name="robot_sn" default="" />
   <xacro:arg name="joint_limits_parameters_file"
@@ -58,4 +66,5 @@
       visual_parameters_file="$(arg visual_parameters_file)"
       arm_prefix="$(arg arm_prefix)"
+      use_sn_prefix="$(arg use_sn_prefix)"
       load_gripper="$(arg load_gripper)"
       gripper_name="$(arg gripper_name)"
@@ -78,4 +87,18 @@
     <xacro:property name="arm_cfg" value="$(find flexiv_description)/config/Enlight-L" />
     <xacro:property name="arm_init_positions" value="${arm_cfg}/initial_positions.yaml" />
+    <!--
+      Per-arm initial positions, overridable independently.
+      Upstream feeds both arms the same file, so a consumer that models only one
+      arm cannot seed a real start pose for it without also moving the other.
+      `initial_positions_file` (the single-arm arg) applies to arm 1, and
+      `initial_positions_file_arm2` to arm 2; each falls back to the vendor
+      default. Only mock hardware reads these (a real arm reports its own
+      joints), so this decides where a simulated arm boots.
+    -->
+    <xacro:arg name="initial_positions_file_arm2" default="" />
+    <xacro:property name="arm1_init_positions"
+      value="${'$(arg initial_positions_file)' if '$(arg initial_positions_file)' != '' else arm_init_positions}" lazy_eval="false" />
+    <xacro:property name="arm2_init_positions"
+      value="${'$(arg initial_positions_file_arm2)' if '$(arg initial_positions_file_arm2)' != '' else arm_init_positions}" lazy_eval="false" />
     <!-- Left arm: owns the shared world link + its base joint. ros2_control handled below. -->
     <xacro:enlight_robot
@@ -86,5 +109,6 @@
       inertia_parameters_file="${arm_cfg}/inertia_parameters.yaml"
       visual_parameters_file="${arm_cfg}/visual_parameters.yaml"
-      arm_prefix="left"
+      arm_prefix="arm1"
+      use_sn_prefix="$(arg use_sn_prefix)"
       load_gripper="$(arg load_gripper)"
       gripper_name="$(arg gripper_name)"
@@ -93,5 +117,5 @@
       use_fake_hardware="$(arg use_fake_hardware)"
       fake_sensor_commands="$(arg fake_sensor_commands)"
-      initial_positions_file="${arm_init_positions}"
+      initial_positions_file="${arm1_init_positions}"
       add_world_link="true"
       create_base_joint="true"
@@ -107,5 +131,6 @@
       inertia_parameters_file="${arm_cfg}/inertia_parameters.yaml"
       visual_parameters_file="${arm_cfg}/visual_parameters.yaml"
-      arm_prefix="right"
+      arm_prefix="arm2"
+      use_sn_prefix="$(arg use_sn_prefix)"
       load_gripper="$(arg load_gripper)"
       gripper_name="$(arg gripper_name)"
@@ -114,5 +139,5 @@
       use_fake_hardware="$(arg use_fake_hardware)"
       fake_sensor_commands="$(arg fake_sensor_commands)"
-      initial_positions_file="${arm_init_positions}"
+      initial_positions_file="${arm2_init_positions}"
       add_world_link="false"
       create_base_joint="true"
@@ -120,15 +145,28 @@
       base_rpy="${radians(right_pose['rx'])} ${radians(right_pose['ry'])} ${radians(right_pose['rz'])}">
     </xacro:enlight_robot>
-    <!-- Single unified ros2_control for both arms (one robot_sn, prefix_left/prefix_right). -->
+    <!--
+      Single unified ros2_control for both arms (one robot_sn,
+      prefix_left/prefix_right).
+      The prefixes are derived the same way `enlight_robot` builds its own, and
+      MUST match it: these become the `<joint name=...>` entries inside
+      `<ros2_control>`, and a name that does not exist in the link/joint tree
+      leaves the controller unable to claim its interfaces. The failure is
+      silent, showing up only as a controller that never reaches `active`.
+      Hardcoding them (as `left_$(arg robot_sn)_`) desyncs the moment
+      `arm_prefix` or `use_sn_prefix` changes.
+    -->
     <xacro:if value="$(arg ros2_control)">
+      <xacro:property name="ll_sn_part" value="${'$(arg robot_sn)' if '$(arg use_sn_prefix)' == 'true' else ''}" lazy_eval="false" />
+      <xacro:property name="ll_prefix_arm1" value="${''.join([part + '_' for part in ['arm1', ll_sn_part] if part != ''])}" />
+      <xacro:property name="ll_prefix_arm2" value="${''.join([part + '_' for part in ['arm2', ll_sn_part] if part != ''])}" />
       <xacro:flexiv_dual_ros2_control
-        prefix_left="left_$(arg robot_sn)_"
-        prefix_right="right_$(arg robot_sn)_"
+        prefix_left="${ll_prefix_arm1}"
+        prefix_right="${ll_prefix_arm2}"
         robot_sn="$(arg robot_sn)"
         rdk_control_mode="$(arg rdk_control_mode)"
         use_fake_hardware="$(arg use_fake_hardware)"
         fake_sensor_commands="$(arg fake_sensor_commands)"
-        initial_positions_file_left="${arm_init_positions}"
-        initial_positions_file_right="${arm_init_positions}" />
+        initial_positions_file_left="${arm1_init_positions}"
+        initial_positions_file_right="${arm2_init_positions}" />
     </xacro:if>
   </xacro:if>
