Commit message: feat: look up joint limits by prefixed joint name
A joint is emitted as `${prefix}jointN` but its limits were read from the
bare `jointN`, so one config file could not describe both arms of a
multi-arm robot, and its keys could not match the joint names the URDF
emits. `get_joint_limits` now prefers the prefixed key and falls back to
the bare one, so every config in `config/` keeps working unchanged and
MICO and Rizon callers are unaffected.

This lets a consumer hold URDF and planning limits in one file: chef
keys its Enlight limits `armN_jointN`, which MoveIt also requires for
`robot_description_planning`.

Co-Authored-By: Claude Opus 5 (1M context) <noreply@anthropic.com>

File: urdf/common/enlight_arm.xacro (robot description, xacro)
@@ -37,5 +37,5 @@
       <xacro:get_kinematics name="joint1" />
       <axis xyz="0 0 1" />
-      <xacro:get_joint_limits name="joint1" />
+      <xacro:get_joint_limits name="joint1" prefix="${prefix}" />
     </joint>
     <joint name="${prefix}joint2" type="revolute">
@@ -44,5 +44,5 @@
       <xacro:get_kinematics name="joint2" />
       <axis xyz="0 0 1" />
-      <xacro:get_joint_limits name="joint2" />
+      <xacro:get_joint_limits name="joint2" prefix="${prefix}" />
     </joint>
     <joint name="${prefix}joint3" type="revolute">
@@ -51,5 +51,5 @@
       <xacro:get_kinematics name="joint3" />
       <axis xyz="0 0 1" />
-      <xacro:get_joint_limits name="joint3" />
+      <xacro:get_joint_limits name="joint3" prefix="${prefix}" />
     </joint>
     <joint name="${prefix}joint4" type="revolute">
@@ -58,5 +58,5 @@
       <xacro:get_kinematics name="joint4" />
       <axis xyz="0 0 1" />
-      <xacro:get_joint_limits name="joint4" />
+      <xacro:get_joint_limits name="joint4" prefix="${prefix}" />
     </joint>
     <joint name="${prefix}joint5" type="revolute">
@@ -65,5 +65,5 @@
       <xacro:get_kinematics name="joint5" />
       <axis xyz="0 0 1" />
-      <xacro:get_joint_limits name="joint5" />
+      <xacro:get_joint_limits name="joint5" prefix="${prefix}" />
     </joint>
     <joint name="${prefix}joint6" type="revolute">
@@ -72,5 +72,5 @@
       <xacro:get_kinematics name="joint6" />
       <axis xyz="0 0 1" />
-      <xacro:get_joint_limits name="joint6" />
+      <xacro:get_joint_limits name="joint6" prefix="${prefix}" />
     </joint>
     <joint name="${prefix}joint7" type="revolute">
@@ -79,5 +79,5 @@
       <xacro:get_kinematics name="joint7" />
       <axis xyz="0 0 1" />
-      <xacro:get_joint_limits name="joint7" />
+      <xacro:get_joint_limits name="joint7" prefix="${prefix}" />
     </joint>
     <joint name="${prefix}link7_to_flange" type="fixed">

File: urdf/common/flexiv_common.xacro (robot description, xacro)
@@ -65,6 +65,12 @@
     name: name of the joint
   -->
-  <xacro:macro name="get_joint_limits" params="name">
-    <xacro:property name="limits" value="${sec_joint_limits[name]}" lazy_eval="false" />
+  <xacro:macro name="get_joint_limits" params="name prefix:=''">
+    <!-- Prefer the prefixed key so one file can hold every arm of a multi-arm
+      robot, and so those keys can match the joint names the URDF emits. Falls
+      back to the bare key, which is how the configs in `config/` are written. -->
+    <xacro:property name="limits_key"
+      value="${prefix + name if (prefix + name) in sec_joint_limits else name}"
+      lazy_eval="false" />
+    <xacro:property name="limits" value="${sec_joint_limits[limits_key]}" lazy_eval="false" />
     <limit lower="${limits['lower']}" upper="${limits['upper']}" effort="${limits['effort']}"
       velocity="${limits['velocity']}" />
